Commit message: Teleop Control

File: ros2_ws/src/unoq_braccio_sim/urdf/braccio.urdf.xacro (robot description, xacro)
@@ -3,4 +3,6 @@
   <xacro:arg name="controllers_file" default=""/>
   <xacro:arg name="mesh_dir" default=""/>
+  <!-- joint_state_publisher_gui only: hide the left finger slider and drive it from "gripper". -->
+  <xacro:arg name="gui_mimic" default="false"/>
   <material name="orange"><color rgba="1.0 0.34 0.02 1"/></material>
   <material name="white"><color rgba="0.86 0.86 0.82 1"/></material>
@@ -168,9 +170,13 @@
   <joint name="left_gripper" type="revolute">
     <axis xyz="0 1 0"/>
-    <!-- Driven as 2.5482 - gripper by joint_trajectory_bridge (mirror of the right finger). -->
-    <limit effort="5" lower="1.2741" upper="2.3732" velocity="2"/>
+    <!-- Driven with the same angle as "gripper" by joint_trajectory_bridge: the flipped
+         frame (pi + 0.2967) and reversed axis make equal angles a mirror image. -->
+    <limit effort="5" lower="0.1750" upper="1.2741" velocity="2"/>
     <origin xyz="-0.010 0 0.03" rpy="0 3.4383 0"/>
     <parent link="wrist_roll_link"/>
     <child link="left_gripper_link"/>
+    <xacro:if value="$(arg gui_mimic)">
+      <mimic joint="gripper" multiplier="1" offset="0"/>
+    </xacro:if>
     <dynamics damping="0.1" friction="0.001"/>
   </joint>

Commit message: gripper gripping friction

File: ros2_ws/src/unoq_braccio_sim/urdf/braccio.urdf.xacro (robot description, xacro)
@@ -162,5 +162,5 @@
   <joint name="gripper" type="revolute">
     <axis xyz="0 -1 0"/>
-    <limit effort="5" lower="0.1750" upper="1.2741" velocity="2"/>
+    <limit effort="1" lower="0.1750" upper="1.2741" velocity="2"/>
     <origin xyz="0.010 0 0.03" rpy="0 -0.2967 0"/>
     <parent link="wrist_roll_link"/>
@@ -172,5 +172,5 @@
     <!-- Driven with the same angle as "gripper" by joint_trajectory_bridge. The flipped
          frame (pi + 0.2967) and reversed axis make equal angles a mirror image. -->
-    <limit effort="5" lower="0.1750" upper="1.2741" velocity="2"/>
+    <limit effort="1" lower="0.1750" upper="1.2741" velocity="2"/>
     <origin xyz="-0.010 0 0.03" rpy="0 3.4383 0"/>
     <parent link="wrist_roll_link"/>
@@ -186,4 +186,8 @@
     <origin xyz="0.03 0 0.055" rpy="0 -1.5708 0"/>
   </joint>
+  <!-- Every joint starts at the "ready" pose (arm straight up, gripper open).
+       Without initial values Gazebo spawns at the URDF zeros, which is servo 180
+       for shoulder, elbow and wrist, so the arm lies across the table and sweeps
+       the cubes away before the controller takes over. -->
   <ros2_control name="GazeboSystem" type="system">
     <hardware>
@@ -192,35 +196,49 @@
     <joint name="base">
       <command_interface name="position"/>
-      <state_interface name="position"/>
+      <state_interface name="position">
+        <param name="initial_value">0.0</param>
+      </state_interface>
       <state_interface name="velocity"/>
     </joint>
     <joint name="shoulder">
       <command_interface name="position"/>
-      <state_interface name="position"/>
+      <state_interface name="position">
+        <param name="initial_value">1.5708</param>
+      </state_interface>
       <state_interface name="velocity"/>
     </joint>
     <joint name="elbow">
       <command_interface name="position"/>
-      <state_interface name="position"/>
+      <state_interface name="position">
+        <param name="initial_value">1.5708</param>
+      </state_interface>
       <state_interface name="velocity"/>
     </joint>
     <joint name="wrist_vertical">
       <command_interface name="position"/>
-      <state_interface name="position"/>
+      <state_interface name="position">
+        <param name="initial_value">1.5708</param>
+      </state_interface>
       <state_interface name="velocity"/>
     </joint>
     <joint name="wrist_rotation">
       <command_interface name="position"/>
-      <state_interface name="position"/>
+      <state_interface name="position">
+        <param name="initial_value">0.0</param>
+      </state_interface>
       <state_interface name="velocity"/>
     </joint>
     <joint name="gripper">
       <command_interface name="position"/>
-      <state_interface name="position"/>
+      <state_interface name="position">
+        <param name="initial_value">0.3399</param>
+      </state_interface>
       <state_interface name="velocity"/>
     </joint>
     <joint name="left_gripper">
       <command_interface name="position"/>
-      <state_interface name="position"/>
+      <state_interface name="position">
+        <param name="initial_value">0.3399</param>
+      </state_interface>
       <state_interface name="velocity"/>
     </joint>
@@ -238,4 +256,13 @@
   <xacro:no_gravity link="left_gripper_link"/>
   <xacro:no_gravity link="camera_link"/>
+  <!-- High-friction finger pads so a squeezed cube does not slide out. -->
+  <xacro:macro name="finger_friction" params="link">
+    <gazebo reference="${link}">
+      <mu1>2.0</mu1>
+      <mu2>2.0</mu2>
+    </gazebo>
+  </xacro:macro>
+  <xacro:finger_friction link="right_gripper_link"/>
+  <xacro:finger_friction link="left_gripper_link"/>
   <!-- Gripper-mounted camera (matches the real Grove Vision AI on the gripper). -->
   <gazebo reference="camera_link">

Commit message: gripper gripping friction

File: ros2_ws/src/unoq_braccio_sim/urdf/braccio.urdf.xacro (robot description, xacro)
@@ -92,7 +92,11 @@
   <link name="right_gripper_link">
     <xacro:mesh_visual filename="braccio_right_gripper.stl" material="white" x="0" y="-0.012" z="0.010" rr="0" rp="1.5708" ry="0"/>
-    <collision>
-      <origin xyz="0.035 -0.012 0.01"/>
-      <geometry><box size="0.08 0.012 0.014"/></geometry>
+    <!-- Straight gripping pad (the visual finger is curved). It sits on the finger
+         plate at the inner edge of the fingertip and is vertical, parallel to the
+         other pad, at servo 90, with the faces 29 mm apart. So a 30 mm cube is
+         squeezed between two flat faces instead of two hooked tips. -->
+    <collision>
+      <origin xyz="0.0836 0 0.0110" rpy="0 -0.2198 0"/>
+      <geometry><box size="0.028 0.012 0.006"/></geometry>
     </collision>
     <xacro:box_inertial mass="0.03" x="0.08" y="0.012" z="0.014"/>
@@ -100,7 +104,8 @@
   <link name="left_gripper_link">
     <xacro:mesh_visual filename="braccio_left_gripper.stl" material="white" x="0" y="-0.012" z="0" rr="0" rp="1.5708" ry="0"/>
-    <collision>
-      <origin xyz="0.035 -0.012 0"/>
-      <geometry><box size="0.08 0.012 0.014"/></geometry>
+    <!-- Mirror of the right finger pad. -->
+    <collision>
+      <origin xyz="0.0836 0 -0.0110" rpy="0 0.2198 0"/>
+      <geometry><box size="0.028 0.012 0.006"/></geometry>
     </collision>
     <xacro:box_inertial mass="0.03" x="0.08" y="0.012" z="0.014"/>

Commit message: attatch detatch joint for cubes

File: ros2_ws/src/unoq_braccio_sim/urdf/braccio.urdf.xacro (robot description, xacro)
@@ -270,4 +270,25 @@
   <xacro:finger_friction link="right_gripper_link"/>
   <xacro:finger_friction link="left_gripper_link"/>
+  <!-- Grasp assist. Finger friction alone does not hold a cube reliably in
+       Gazebo, so a grasped cube is welded to the wrist with a DetachableJoint
+       and let go on release (sim_grasp_attacher drives the topics; names must
+       match braccio_workspace.grasp_topic). Note: in Gazebo Harmonic every
+       DetachableJoint attaches as soon as the robot spawns; sim_grasp_attacher
+       detaches them all straight away. -->
+  <xacro:macro name="cube_grasp" params="color">
+    <gazebo>
+      <plugin filename="gz-sim-detachable-joint-system" name="gz::sim::systems::DetachableJoint">
+        <parent_link>wrist_roll_link</parent_link>
+        <child_model>${color}_cube</child_model>
+        <child_link>link</child_link>
+        <attach_topic>/sim/grasp/${color}_cube/attach</attach_topic>
+        <detach_topic>/sim/grasp/${color}_cube/detach</detach_topic>
+        <output_topic>/sim/grasp/${color}_cube/state</output_topic>
+      </plugin>
+    </gazebo>
+  </xacro:macro>
+  <xacro:cube_grasp color="red"/>
+  <xacro:cube_grasp color="blue"/>
+  <xacro:cube_grasp color="yellow"/>
   <!-- Gripper-mounted camera (matches the real Grove Vision AI on the gripper). -->
   <gazebo reference="camera_link">
